File: hardware/KiCAD/cellSymphony.kicad_pcb (KiCad board)
At the start: 2 copper layers, 56.5 x 151 mm, 11 parts, among them SW1 RotaryEncoder_Switch, SW2 RotaryEncoder_Switch, SW3 RotaryEncoder_Switch, SW4 RotaryEncoder_Switch, SW5 RotaryEncoder_Switch, U1 Raspberry Pi Zero 2 W

Commit message: Midi full implementation, cleanup
Parts:
- ADA4090, ADA6250, U1: moved to B.Cu
- moved U1 3.23 mm to (46.5, 133.5), turned to 90 degrees
- turned ADA4090 to 180 degrees
- turned ADA6250 to 180 degrees
Routing:
- net Net-(OLED1-VIN): track 84.6 -> 136.2 mm
- net Net-(U1-GPIO20): track 107.0 -> 61.4 mm, vias 1 -> 0
- net Net-(U1-GPIO26): track 71.1 -> 27.9 mm
- net Net-(U1-GPIO16): track 93.9 -> 52.4 mm, vias 1 -> 0
- net Net-(U1-GPIO4/GPIO_GCLK): track 50.3 -> 89.6 mm
- net Net-(U1-GPIO13): track 91.0 -> 57.1 mm, vias 1 -> 0
- net Net-(U1-GPIO14/TXD0): track 27.1 -> 59.9 mm
- net Net-(NeoKey1-SDA): track 36.0 -> 65.1 mm
- net Net-(U1-GPIO12): track 123.5 -> 95.6 mm, vias 0 -> 1
- net Net-(NeoKey1-SCL): track 34.3 -> 60.9 mm
- net Net-(U1-GPIO17/GPIO_GEN0): track 73.5 -> 96.4 mm
- net Net-(U1-GPIO6): track 107.7 -> 85.3 mm
- net Net-(U1-GPIO5): track 109.8 -> 88.0 mm, vias 1 -> 0
- net Net-(GY-PCM5102-DIN): track 27.1 -> 46.9 mm, vias 0 -> 4
- net Net-(U1-GPIO27/GPIO_GEN2): track 56.2 -> 75.9 mm
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